File: ws2812-stm32-interface.kicad_pcb (KiCad board)
At the start: 2 copper layers, 14 parts, among them J1 Conn_01x03, J2 Conn_01x03, U1 74AHCT1G125

Commit message: update,
Parts:
- moved R2 1.00 mm to (37.8, 26.6)
- moved D2 0.50 mm to (39.2, 19.5)
Routing:
- net VCC: track 44.8 -> 46.4 mm
- net /PWM_TO_LED: track 42.8 -> 41.8 mm
- net Net-(D4-Pad2): track 3.75 -> 2.75 mm
- added copper zone on B.Cu, net GND
- added copper zone on F.Cu, net GND
Other:
- board outline added: 33 x 21.2 mm
Changed lines of the file:
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@@
   (general
     (thickness 1.6)
-    (drawings 0)
-    (tracks 75)
+    (drawings 4)
+    (tracks 76)
     (zones 0)
     (modules 14)
@@
     (descr "simple 4-pin terminal block, pitch 5.08mm, revamped version of bornier4")
     (tags "terminal block bornier4")
-    (fp_text reference J2 (at 7.6 -4.8 90) (layer F.SilkS)
+    (fp_text reference J2 (at -1.75 -4.75 90) (layer F.SilkS)
       (effects (font (size 1 1) (thickness 0.15)))
     )
@@
   )
   (module Diodes_SMD:D_SOD-123F (layer F.Cu)
-    (at 38.75 19.5)
+    (at 39.25 19.5)
     (descr D_SOD-123F)
     (tags D_SOD-123F)
     (attr smd)
-    (fp_text reference D2 (at -0.127 -1.905) (layer F.SilkS)
+    (fp_text reference D2 (at 0 2) (layer F.SilkS)
       (effects (font (size 1 1) (thickness 0.15)))
     )
@@
     (tags "resistor 0805")
     (attr smd)
-    (fp_text reference D4 (at 0 -1.7 270) (layer F.SilkS)
+    (fp_text reference D4 (at 3.65 0 270) (layer F.SilkS)
       (effects (font (size 1 1) (thickness 0.15)))
     )
@@
     (tags "resistor 0805")
     (attr smd)
-    (fp_text reference D3 (at 0 -1.7 270) (layer F.SilkS)
+    (fp_text reference D3 (at 3.6 0 270) (layer F.SilkS)
       (effects (font (size 1 1) (thickness 0.15)))
     )
@@
   )
   (module Resistors_SMD:R_0805_HandSoldering (layer F.Cu)
-    (at 38.75 26.6 270)
+    (at 37.75 26.6 270)
     (descr "Resistor SMD 0805, hand soldering")
     (tags "resistor 0805")
     (attr smd)
-    (fp_text reference R2 (at 0 -1.7 270) (layer F.SilkS)
+    (fp_text reference R2 (at 3.65 0 270) (layer F.SilkS)
       (effects (font (size 1 1) (thickness 0.15)))
     )
@@
     (tags "resistor 0805")
     (attr smd)
-    (fp_text reference R1 (at 0 -1.7 270) (layer F.SilkS)
+    (fp_text reference R1 (at 3.6 0 270) (layer F.SilkS)
       (effects (font (size 1 1) (thickness 0.15)))
     )
@@
     (tags "SOT-23-5 hand-soldering")
     (attr smd)
-    (fp_text reference U1 (at 0 -2.9 270) (layer F.SilkS)
+    (fp_text reference U1 (at 3.25 0 270) (layer F.SilkS)
       (effects (font (size 1 1) (thickness 0.15)))
     )
@@
     (descr "Through hole straight pin header, 1x03, 2.54mm pitch, single row")
     (tags "Through hole pin header THT 1x03 2.54mm single row")
-    (fp_text reference J1 (at 0 -2.33 270) (layer F.SilkS)
+    (fp_text reference J1 (at 2.5 5.75 270) (layer F.SilkS)
       (effects (font (size 1 1) (thickness 0.15)))
     )
@@
     )
   )
+  (gr_line (start 52.75 12.75) (end 19.75 12.75) (layer Edge.Cuts) (width 0.15))
+  (gr_line (start 52.75 34) (end 52.75 12.75) (layer Edge.Cuts) (width 0.15))
+  (gr_line (start 19.75 34) (end 52.75 34) (layer Edge.Cuts) (width 0.15))
+  (gr_line (start 19.75 12.75) (end 19.75 34) (layer Edge.Cuts) (width 0.15))
   (segment (start 21.92 15) (end 21.92 16.67) (width 0.5) (layer F.Cu) (net 1))
   (segment (start 21.92 16.67) (end 23.25 18) (width 0.5) (layer F.Cu) (net 1))
@@
   (segment (start 36.337702 16.612568) (end 39.587702 16.612568) (width 1) (layer F.Cu) (net 4))
   (segment (start 39.587702 16.612568) (end 42.837702 16.612568) (width 1) (layer F.Cu) (net 4))
-  (segment (start 36.337702 16.612568) (end 36.337702 19.087702) (width 1) (layer F.Cu) (net 4))
-  (segment (start 37.35 20.1) (end 37.35 21.75) (width 1) (layer F.Cu) (net 4))
-  (segment (start 36.337702 19.087702) (end 37.35 20.1) (width 1) (layer F.Cu) (net 4))
-  (segment (start 37.35 23.85) (end 38.75 25.25) (width 1) (layer F.Cu) (net 4))
-  (segment (start 37.35 21.75) (end 37.35 23.85) (width 1) (layer F.Cu) (net 4))
   (segment (start 29.887432 16.612568) (end 30.337702 16.612568) (width 1) (layer F.Cu) (net 4))
   (segment (start 27 19.5) (end 29.887432 16.612568) (width 1) (layer F.Cu) (net 4))
@@
   (segment (start 26.4 23.1) (end 27 22.5) (width 1) (layer F.Cu) (net 4))
   (segment (start 34 19.5) (end 37.35 19.5) (width 1) (layer F.Cu) (net 4))
-  (segment (start 47.58 25.25) (end 48.25 25.92) (width 1) (layer F.Cu) (net 4))
-  (segment (start 38.75 25.25) (end 47.58 25.25) (width 1) (layer F.Cu) (net 4))
+  (segment (start 48.25 25.92) (end 40.67 25.92) (width 1) (layer F.Cu) (net 4))
+  (segment (start 40 25.25) (end 38.75 25.25) (width 1) (layer F.Cu) (net 4))
+  (segment (start 40 25.25) (end 40.67 25.92) (width 1) (layer F.Cu) (net 4))
+  (segment (start 37.75 25.25) (end 40 25.25) (width 1) (layer F.Cu) (net 4))
+  (segment (start 37.75 19.6) (end 37.85 19.5) (width 1) (layer F.Cu) (net 4))
+  (segment (start 37.75 25.25) (end 37.75 19.6) (width 1) (layer F.Cu) (net 4))
+  (segment (start 34 17.274866) (end 33.337702 16.612568) (width 1) (layer F.Cu) (net 4))
+  (segment (start 34 19.5) (end 34 17.274866) (width 1) (layer F.Cu) (net 4))
   (via (at 23.25 26.75) (size 1.2) (drill 0.4) (layers F.Cu B.Cu) (net 5))
-  (segment (start 23.25 23.15) (end 23.3 23.1) (width 0.5) (layer F.Cu) (net 5))
-  (segment (start 23.25 26.75) (end 23.25 23.15) (width 0.5) (layer F.Cu) (net 5))
-  (segment (start 23.25 31) (end 23.25 26.75) (width 0.5) (layer B.Cu) (net 5))
-  (segment (start 48.25 20.84) (end 45.41 20.84) (width 0.5) (layer B.Cu) (net 5))
-  (segment (start 45.41 20.84) (end 43.5 22.75) (width 0.5) (layer B.Cu) (net 5))
-  (segment (start 43.5 22.75) (end 43.5 31) (width 0.5) (layer B.Cu) (net 5))
-  (segment (start 43.5 31) (end 42.5 32) (width 0.5) (layer B.Cu) (net 5))
-  (segment (start 42.5 32) (end 24.25 32) (width 0.5) (layer B.Cu) (net 5))
-  (segment (start 24.25 32) (end 23.25 31) (width 0.5) (layer B.Cu) (net 5))
+  (segment (start 45.91 20.84) (end 43 23.75) (width 0.5) (layer B.Cu) (net 5))
+  (segment (start 48.25 20.84) (end 45.91 20.84) (width 0.5) (layer B.Cu) (net 5))
+  (segment (start 43 23.75) (end 43 30.5) (width 0.5) (layer B.Cu) (net 5))
+  (segment (start 43 30.5) (end 41.5 32) (width 0.5) (layer B.Cu) (net 5))
+  (segment (start 23.3 26.7) (end 23.25 26.75) (width 0.5) (layer F.Cu) (net 5))
+  (segment (start 23.3 23.1) (end 23.3 26.7) (width 0.5) (layer F.Cu) (net 5))
+  (segment (start 23.25 30.75) (end 24.5 32) (width 0.5) (layer B.Cu) (net 5))
+  (segment (start 23.25 26.75) (end 23.25 30.75) (width 0.5) (layer B.Cu) (net 5))
+  (segment (start 41.5 32) (end 24.5 32) (width 0.5) (layer B.Cu) (net 5))
   (segment (start 29.75 28) (end 32.25 28) (width 0.25) (layer F.Cu) (net 6))
-  (segment (start 35 27.95) (end 38.75 27.95) (width 0.25) (layer F.Cu) (net 7))
+  (segment (start 35 27.95) (end 37.75 27.95) (width 0.25) (layer F.Cu) (net 7))
   (segment (start 40.15 19.5) (end 44.25 19.5) (width 1) (layer F.Cu) (net 8))
   (segment (start 44.25 19.5) (end 45.5 18.25) (width 1) (layer F.Cu) (net 8))
@@
   (segment (start 51.25 28) (end 48.25 31) (width 1) (layer F.Cu) (net 8))
   (segment (start 51.25 19.25) (end 51.25 28) (width 1) (layer F.Cu) (net 8))
+  (zone (net 3) (net_name GND) (layer F.Cu) (hatch edge 0.508)
+    (connect_pads (clearance 0.508))
+    (min_thickness 0.254)
+    (fill yes (arc_segments 16) (thermal_gap 0.508) (thermal_bridge_width 0.508))
+    (polygon
+      (pts
+        (xy 20 13) (xy 20 33.75) (xy 52.5 33.75) (xy 52.5 13)
+      )
+    )
+  )
+  (zone (net 3) (net_name GND) (layer B.Cu) (hatch edge 0.508)
+    (connect_pads (clearance 0.508))
+    (min_thickness 0.254)
+    (fill yes (arc_segments 16) (thermal_gap 0.508) (thermal_bridge_width 0.508))
+    (polygon
+      (pts
+        (xy 20 13) (xy 20 33.75) (xy 52.5 33.75) (xy 52.5 13)
+      )
+    )
+  )
 )

Commit message: update,
Parts:
- D1, D2: value mbr120 -> MBR120
- D3: value LED -> GREEN
- D4: value LED -> RED
Routing:
- net GND: vias 2 -> 3
Other:
- board text added: "WS2812-CONTROL REV 1.0"
Changed lines of the file:
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@@
   (general
     (thickness 1.6)
-    (drawings 4)
-    (tracks 76)
+    (drawings 5)
+    (tracks 77)
     (zones 0)
     (modules 14)
@@
       (outputformat 1)
       (mirror false)
-      (drillshape 1)
+      (drillshape 0)
       (scaleselection 1)
-      (outputdirectory ""))
+      (outputdirectory "gerber/"))
   )
   (net 0 "")
@@
       (effects (font (size 1 1) (thickness 0.15)))
     )
-    (fp_text value mbr120 (at 0 2.1) (layer F.Fab)
+    (fp_text value MBR120 (at 0 2.1) (layer F.Fab)
       (effects (font (size 1 1) (thickness 0.15)))
     )
@@
       (effects (font (size 1 1) (thickness 0.15)))
     )
-    (fp_text value mbr120 (at 0 2.1 180) (layer F.Fab)
+    (fp_text value MBR120 (at 0 2.1 180) (layer F.Fab)
       (effects (font (size 1 1) (thickness 0.15)))
     )
@@
       (effects (font (size 1 1) (thickness 0.15)))
     )
-    (fp_text value LED (at 0 1.75 270) (layer F.Fab)
+    (fp_text value RED (at 0 1.75 270) (layer F.Fab)
       (effects (font (size 1 1) (thickness 0.15)))
     )
@@
       (effects (font (size 1 1) (thickness 0.15)))
     )
-    (fp_text value LED (at 0 1.75 270) (layer F.Fab)
+    (fp_text value GREEN (at 0 1.75 270) (layer F.Fab)
       (effects (font (size 1 1) (thickness 0.15)))
     )
@@
       (rotate (xyz 0 0 0))
     )
+  )
+  (gr_text "WS2812-CONTROL REV 1.0" (at 20.5 32.5) (layer F.SilkS)
+    (effects (font (size 1 1) (thickness 0.25)) (justify left))
   )
   (gr_line (start 52.75 12.75) (end 19.75 12.75) (layer Edge.Cuts) (width 0.15))
@@
   (segment (start 23.124999 20.5) (end 23.224999 20.4) (width 0.5) (layer F.Cu) (net 3))
   (segment (start 21.25 20.5) (end 23.124999 20.5) (width 1) (layer F.Cu) (net 3))
+  (via (at 40.5 23) (size 0.8) (drill 0.4) (layers F.Cu B.Cu) (net 3))
   (segment (start 30.337702 16.612568) (end 33.337702 16.612568) (width 1) (layer F.Cu) (net 4))
   (segment (start 33.337702 16.612568) (end 36.337702 16.612568) (width 1) (layer F.Cu) (net 4))

Commit message: update,
Parts:
- moved D2 11.0 mm to (42.5, 30.0), turned to 270 degrees
Routing:
- net V_EXT_LED: track 25.0 -> 5.92 mm
- net VCC: track 46.4 -> 55.2 mm, vias 0 -> 1
- net /PWM_TO_LED: track 41.8 -> 39.9 mm, vias 1 -> 0
Changed lines of the file:
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@@
     (thickness 1.6)
     (drawings 5)
-    (tracks 77)
+    (tracks 76)
     (zones 0)
     (modules 14)
@@
   )
   (module Diodes_SMD:D_SOD-123F (layer F.Cu)
-    (at 39.25 19.5)
+    (at 42.5 30 270)
     (descr D_SOD-123F)
     (tags D_SOD-123F)
     (attr smd)
-    (fp_text reference D2 (at 0 2) (layer F.SilkS)
-      (effects (font (size 1 1) (thickness 0.15)))
-    )
-    (fp_text value MBR120 (at 0 2.1) (layer F.Fab)
-      (effects (font (size 1 1) (thickness 0.15)))
-    )
-    (fp_text user %R (at -0.127 -1.905) (layer F.Fab)
+    (fp_text reference D2 (at 0 2 270) (layer F.SilkS)
+      (effects (font (size 1 1) (thickness 0.15)))
+    )
+    (fp_text value MBR120 (at 0 2.1 270) (layer F.Fab)
+      (effects (font (size 1 1) (thickness 0.15)))
+    )
+    (fp_text user %R (at -0.127 -1.905 270) (layer F.Fab)
       (effects (font (size 1 1) (thickness 0.15)))
     )
@@
     (fp_line (start -2.2 1) (end 1.65 1) (layer F.SilkS) (width 0.12))
     (fp_line (start -2.2 -1) (end 1.65 -1) (layer F.SilkS) (width 0.12))
-    (pad 1 smd rect (at -1.4 0) (size 1.1 1.1) (layers F.Cu F.Paste F.Mask)
-      (net 4 VCC))
-    (pad 2 smd rect (at 1.4 0) (size 1.1 1.1) (layers F.Cu F.Paste F.Mask)
+    (pad 1 smd rect (at -1.4 0 270) (size 1.1 1.1) (layers F.Cu F.Paste F.Mask)
+      (net 4 VCC))
+    (pad 2 smd rect (at 1.4 0 270) (size 1.1 1.1) (layers F.Cu F.Paste F.Mask)
       (net 8 V_EXT_LED))
     (model ${KISYS3DMOD}/Diodes_SMD.3dshapes/D_SOD-123F.wrl
@@
   (segment (start 23.124999 20.5) (end 23.224999 20.4) (width 0.5) (layer F.Cu) (net 3))
   (segment (start 21.25 20.5) (end 23.124999 20.5) (width 1) (layer F.Cu) (net 3))
-  (via (at 40.5 23) (size 0.8) (drill 0.4) (layers F.Cu B.Cu) (net 3))
+  (via (at 38 20) (size 2) (drill 0.4) (layers F.Cu B.Cu) (net 3))
   (segment (start 30.337702 16.612568) (end 33.337702 16.612568) (width 1) (layer F.Cu) (net 4))
   (segment (start 33.337702 16.612568) (end 36.337702 16.612568) (width 1) (layer F.Cu) (net 4))
@@
   (segment (start 25.2 23.1) (end 26.4 23.1) (width 1) (layer F.Cu) (net 4))
   (segment (start 26.4 23.1) (end 27 22.5) (width 1) (layer F.Cu) (net 4))
-  (segment (start 34 19.5) (end 37.35 19.5) (width 1) (layer F.Cu) (net 4))
-  (segment (start 48.25 25.92) (end 40.67 25.92) (width 1) (layer F.Cu) (net 4))
-  (segment (start 40 25.25) (end 38.75 25.25) (width 1) (layer F.Cu) (net 4))
-  (segment (start 40 25.25) (end 40.67 25.92) (width 1) (layer F.Cu) (net 4))
-  (segment (start 37.75 25.25) (end 40 25.25) (width 1) (layer F.Cu) (net 4))
-  (segment (start 37.75 19.6) (end 37.85 19.5) (width 1) (layer F.Cu) (net 4))
-  (segment (start 37.75 25.25) (end 37.75 19.6) (width 1) (layer F.Cu) (net 4))
   (segment (start 34 17.274866) (end 33.337702 16.612568) (width 1) (layer F.Cu) (net 4))
   (segment (start 34 19.5) (end 34 17.274866) (width 1) (layer F.Cu) (net 4))
-  (via (at 23.25 26.75) (size 1.2) (drill 0.4) (layers F.Cu B.Cu) (net 5))
-  (segment (start 45.91 20.84) (end 43 23.75) (width 0.5) (layer B.Cu) (net 5))
-  (segment (start 48.25 20.84) (end 45.91 20.84) (width 0.5) (layer B.Cu) (net 5))
-  (segment (start 43 23.75) (end 43 30.5) (width 0.5) (layer B.Cu) (net 5))
-  (segment (start 43 30.5) (end 41.5 32) (width 0.5) (layer B.Cu) (net 5))
-  (segment (start 23.3 26.7) (end 23.25 26.75) (width 0.5) (layer F.Cu) (net 5))
-  (segment (start 23.3 23.1) (end 23.3 26.7) (width 0.5) (layer F.Cu) (net 5))
-  (segment (start 23.25 30.75) (end 24.5 32) (width 0.5) (layer B.Cu) (net 5))
-  (segment (start 23.25 26.75) (end 23.25 30.75) (width 0.5) (layer B.Cu) (net 5))
-  (segment (start 41.5 32) (end 24.5 32) (width 0.5) (layer B.Cu) (net 5))
-  (segment (start 29.75 28) (end 32.25 28) (width 0.25) (layer F.Cu) (net 6))
-  (segment (start 35 27.95) (end 37.75 27.95) (width 0.25) (layer F.Cu) (net 7))
-  (segment (start 40.15 19.5) (end 44.25 19.5) (width 1) (layer F.Cu) (net 8))
-  (segment (start 44.25 19.5) (end 45.5 18.25) (width 1) (layer F.Cu) (net 8))
-  (segment (start 45.5 18.25) (end 50.25 18.25) (width 1) (layer F.Cu) (net 8))
-  (segment (start 50.25 18.25) (end 51.25 19.25) (width 1) (layer F.Cu) (net 8))
-  (segment (start 51.25 28) (end 48.25 31) (width 1) (layer F.Cu) (net 8))
-  (segment (start 51.25 19.25) (end 51.25 28) (width 1) (layer F.Cu) (net 8))
+  (via (at 35.5 22.75) (size 2) (drill 0.4) (layers F.Cu B.Cu) (net 4))
+  (segment (start 48.25 25.92) (end 38.67 25.92) (width 1) (layer B.Cu) (net 4))
+  (segment (start 38.67 25.92) (end 35.5 22.75) (width 1) (layer B.Cu) (net 4))
+  (segment (start 34 21.25) (end 34 19.5) (width 1) (layer F.Cu) (net 4))
+  (segment (start 35.5 22.75) (end 34 21.25) (width 1) (layer F.Cu) (net 4))
+  (segment (start 37.75 25.25) (end 37.75 23.5) (width 1) (layer F.Cu) (net 4))
+  (segment (start 37 22.75) (end 35.5 22.75) (width 1) (layer F.Cu) (net 4))
+  (segment (start 37.75 23.5) (end 37 22.75) (width 1) (layer F.Cu) (net 4))
+  (segment (start 43.43 25.92) (end 42.5 26.85) (width 1) (layer F.Cu) (net 4))
+  (segment (start 48.25 25.92) (end 43.43 25.92) (width 1) (layer F.Cu) (net 4))
+  (segment (start 42.5 26.85) (end 42.5 28.44999) (width 1) (layer F.Cu) (net 4))
+  (segment (start 43.91 20.84) (end 48.25 20.84) (width 0.5) (layer F.Cu) (net 5))
+  (segment (start 23.3 29.3) (end 25 31) (width 0.5) (layer F.Cu) (net 5))
+  (segment (start 23.3 23.1) (end 23.3 29.3) (width 0.5) (layer F.Cu) (net 5))
+  (segment (start 25 31) (end 38.75 31) (width 0.5) (layer F.Cu) (net 5))
+  (segment (start 42.41 20.84) (end 43.91 20.84) (width 0.5) (layer F.Cu) (net 5))
+  (segment (start 38.75 31) (end 40.25 29.5) (width 0.5) (layer F.Cu) (net 5))
+  (segment (start 40.25 29.5) (end 40.25 23) (width 0.5) (layer F.Cu) (net 5))
+  (segment (start 40.25 23) (end 42.41 20.84) (width 0.5) (layer F.Cu) (net 5))
+  (segment (start 29.75 28) (end 32.25 28) (width 0.4) (layer F.Cu) (net 6))
+  (segment (start 35 27.95) (end 37.75 27.95) (width 0.4) (layer F.Cu) (net 7))
+  (segment (start 48.25 31) (end 45.25 31) (width 1) (layer F.Cu) (net 8))
+  (segment (start 44.85 31.4) (end 42.5 31.4) (width 1) (layer F.Cu) (net 8))
+  (segment (start 45.25 31) (end 44.85 31.4) (width 1) (layer F.Cu) (net 8))
   (zone (net 3) (net_name GND) (layer F.Cu) (hatch edge 0.508)
     (connect_pads (clearance 0.508))

Commit message: update,
Parts:
- moved U1 5.50 mm to (24.2, 27.2)
- moved J1 4.01 mm to (23.0, 15.2), turned to 0 degrees
Routing:
- net GND: track 60.7 -> 68.0 mm, vias 3 -> 1
- net VCC: track 55.2 -> 61.4 mm
- net /PWM_TO_LED: track 39.9 -> 37.7 mm
- net +5V: track 16.0 -> 14.8 mm
- net /MCU_LED_PWM: track 6.66 -> 7.40 mm
