File: ws2812-stm32-interface.kicad_pcb (KiCad board)
At the start: 2 copper layers, 100.3 x 76.2 mm, 81 parts, among them J1 Conn_01x03, J2 Conn_01x03, J3 WS2812_DEST, J4 WS2812_SOURCE, U1 74AHCT1G125

Commit message: update,
Routing:
- net Net-(J4-Pad3): track 36.8 -> 35.1 mm
Changed lines of the file:
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@@
   (segment (start 42.921761 41.384571) (end 43.14676 41.60957) (width 0.5) (layer F.Cu) (net 3) (status 30))
   (segment (start 32.49676 43.884571) (end 32.49676 41.384571) (width 1) (layer F.Cu) (net 3) (status 10))
-  (via (at 47.49676 38.634571) (size 2) (drill 0.4) (layers F.Cu B.Cu) (net 3))
   (via (at 58.928 18.288) (size 2) (drill 0.4) (layers F.Cu B.Cu) (net 3))
   (segment (start 58.928 18.288) (end 58.928 16.256) (width 1) (layer B.Cu) (net 3))
@@
   (segment (start 37.846 46.134571) (end 39.99676 46.134571) (width 1) (layer F.Cu) (net 3))
   (segment (start 33.24676 46.134571) (end 37.846 46.134571) (width 1) (layer F.Cu) (net 3))
+  (via (at 49.022 34.544) (size 2) (drill 0.4) (layers F.Cu B.Cu) (net 3))
   (segment (start 33.859328 36.546869) (end 33.859328 33.546869) (width 1) (layer F.Cu) (net 4) (status 30))
   (segment (start 33.859328 33.546869) (end 33.859328 30.546869) (width 1) (layer F.Cu) (net 4) (status 30))
@@
   (segment (start 45.212 26.634571) (end 50.581429 26.634571) (width 0.5) (layer F.Cu) (net 5))
   (segment (start 40.24676 26.634571) (end 45.212 26.634571) (width 0.5) (layer F.Cu) (net 5))
-  (segment (start 49.04676 43.584571) (end 45.84676 43.584571) (width 0.5) (layer F.Cu) (net 5))
-  (segment (start 49.49676 43.134571) (end 49.04676 43.584571) (width 0.5) (layer F.Cu) (net 5))
   (segment (start 45.212 26.634571) (end 49.49676 26.634571) (width 0.5) (layer F.Cu) (net 5))
-  (segment (start 49.49676 35.56) (end 49.49676 35.52676) (width 0.5) (layer F.Cu) (net 5))
-  (segment (start 49.49676 35.56) (end 49.49676 43.134571) (width 0.5) (layer F.Cu) (net 5))
-  (segment (start 49.49676 35.52676) (end 48.26 34.29) (width 0.5) (layer F.Cu) (net 5))
-  (segment (start 48.26 34.29) (end 48.26 26.67) (width 0.5) (layer F.Cu) (net 5))
   (segment (start 40.282189 26.67) (end 38.08676 24.474571) (width 0.5) (layer F.Cu) (net 5))
   (segment (start 50.8 26.67) (end 40.282189 26.67) (width 0.5) (layer F.Cu) (net 5))
+  (segment (start 46.99 26.67) (end 48.26 26.67) (width 0.5) (layer F.Cu) (net 5))
+  (segment (start 46.99 39.624) (end 46.99 26.67) (width 0.5) (layer F.Cu) (net 5))
+  (segment (start 48.26 40.894) (end 46.99 39.624) (width 0.5) (layer F.Cu) (net 5))
+  (segment (start 48.26 42.926) (end 48.26 40.894) (width 0.5) (layer F.Cu) (net 5))
+  (segment (start 45.84676 43.584571) (end 47.601429 43.584571) (width 0.5) (layer F.Cu) (net 5))
+  (segment (start 47.601429 43.584571) (end 48.26 42.926) (width 0.5) (layer F.Cu) (net 5))
   (segment (start 84.077713 19.888) (end 82.372 19.888) (width 0.25) (layer F.Cu) (net 6))
   (segment (start 82.372 19.888) (end 81.788 19.304) (width 0.25) (layer F.Cu) (net 6))
@@
   (segment (start 116.727426 52.39314) (end 118.43314 52.39314) (width 0.25) (layer F.Cu) (net 18))
   (segment (start 118.43314 52.39314) (end 118.872 52.832) (width 0.25) (layer F.Cu) (net 18))
-  (segment (start 125.944 53.808) (end 125.944 52.39314) (width 0.25) (layer F.Cu) (net 19))
+  (segment (start 55.118 58.42) (end 125.984 58.42) (width 0.25) (layer F.Cu) (net 19))
+  (segment (start 125.984 58.42) (end 127.508 56.896) (width 0.25) (layer F.Cu) (net 19))
+  (segment (start 54.102 59.436) (end 55.118 58.42) (width 0.25) (layer F.Cu) (net 19))
+  (segment (start 54.102 63.757425) (end 54.102 59.436) (width 0.25) (layer F.Cu) (net 19))
+  (segment (start 56.428 64.519425) (end 54.864 64.519425) (width 0.25) (layer F.Cu) (net 19))
+  (segment (start 54.864 64.519425) (end 54.102 63.757425) (width 0.25) (layer F.Cu) (net 19))
+  (segment (start 127.508 56.896) (end 127.508 54.61) (width 0.25) (layer F.Cu) (net 19))
   (segment (start 127 54.102) (end 126.238 54.102) (width 0.25) (layer F.Cu) (net 19))
   (segment (start 127.508 54.61) (end 127 54.102) (width 0.25) (layer F.Cu) (net 19))
-  (segment (start 127.508 56.896) (end 127.508 54.61) (width 0.25) (layer F.Cu) (net 19))
-  (segment (start 56.428 64.519425) (end 54.864 64.519425) (width 0.25) (layer F.Cu) (net 19))
   (segment (start 126.238 54.102) (end 125.944 53.808) (width 0.25) (layer F.Cu) (net 19))
-  (segment (start 54.102 59.436) (end 55.118 58.42) (width 0.25) (layer F.Cu) (net 19))
-  (segment (start 54.864 64.519425) (end 54.102 63.757425) (width 0.25) (layer F.Cu) (net 19))
-  (segment (start 54.102 63.757425) (end 54.102 59.436) (width 0.25) (layer F.Cu) (net 19))
-  (segment (start 55.118 58.42) (end 125.984 58.42) (width 0.25) (layer F.Cu) (net 19))
-  (segment (start 125.984 58.42) (end 127.508 56.896) (width 0.25) (layer F.Cu) (net 19))
+  (segment (start 125.944 53.808) (end 125.944 52.39314) (width 0.25) (layer F.Cu) (net 19))
   (segment (start 61.428 61.319425) (end 63.097425 61.319425) (width 0.25) (layer F.Cu) (net 20))
   (segment (start 63.097425 61.319425) (end 63.5 61.722) (width 0.25) (layer F.Cu) (net 20))
@@
   (segment (start 126.492 22.352) (end 127.508 21.336) (width 0.25) (layer F.Cu) (net 53))
   (segment (start 55.118 22.352) (end 126.492 22.352) (width 0.25) (layer F.Cu) (net 53))
-  (segment (start 116.727426 16.688) (end 116.727426 17.667426) (width 0.25) (layer F.Cu) (net 54))
-  (segment (start 116.727426 17.667426) (end 117.348 18.288) (width 0.25) (layer F.Cu) (net 54))
-  (segment (start 117.348 18.288) (end 120.396 18.288) (width 0.25) (layer F.Cu) (net 54))
-  (segment (start 120.944 18.836) (end 120.944 19.888) (width 0.25) (layer F.Cu) (net 54))
-  (segment (start 120.396 18.288) (end 120.944 18.836) (width 0.25) (layer F.Cu) (net 54))
-  (segment (start 107.510855 16.688) (end 107.510855 17.594855) (width 0.25) (layer F.Cu) (net 55))
-  (segment (start 107.510855 17.594855) (end 108.204 18.288) (width 0.25) (layer F.Cu) (net 55))
-  (segment (start 108.204 18.288) (end 111.252 18.288) (width 0.25) (layer F.Cu) (net 55))
-  (segment (start 111.727426 18.763426) (end 111.727426 19.888) (width 0.25) (layer F.Cu) (net 55))
-  (segment (start 111.252 18.288) (end 111.727426 18.763426) (width 0.25) (layer F.Cu) (net 55))
+  (segment (start 116.727426 16.688) (end 118.288 16.688) (width 0.25) (layer F.Cu) (net 54))
+  (segment (start 118.288 16.688) (end 118.872 17.272) (width 0.25) (layer F.Cu) (net 54))
+  (segment (start 118.872 17.272) (end 118.872 19.558) (width 0.25) (layer F.Cu) (net 54))
+  (segment (start 119.202 19.888) (end 120.944 19.888) (width 0.25) (layer F.Cu) (net 54))
+  (segment (start 118.872 19.558) (end 119.202 19.888) (width 0.25) (layer F.Cu) (net 54))
+  (segment (start 107.510855 16.688) (end 109.398 16.688) (width 0.25) (layer F.Cu) (net 55))
+  (segment (start 109.398 16.688) (end 109.728 17.018) (width 0.25) (layer F.Cu) (net 55))
+  (segment (start 110.312 19.888) (end 109.728 19.304) (width 0.25) (layer F.Cu) (net 55))
+  (segment (start 111.727426 19.888) (end 110.312 19.888) (width 0.25) (layer F.Cu) (net 55))
+  (segment (start 109.728 17.018) (end 109.728 19.304) (width 0.25) (layer F.Cu) (net 55))
   (segment (start 102.510855 19.888) (end 100.66 19.888) (width 0.25) (layer F.Cu) (net 56))
   (segment (start 100.66 19.888) (end 100.076 19.304) (width 0.25) (layer F.Cu) (net 56))
@@
   (segment (start 52.07 29.21) (end 52.578 29.21) (width 0.25) (layer F.Cu) (net 73))
   (segment (start 52.578 29.21) (end 53.086 28.702) (width 0.25) (layer F.Cu) (net 73))
-  (segment (start 50.8 54.102) (end 50.8 31.75) (width 0.25) (layer F.Cu) (net 74))
-  (segment (start 46.482 58.42) (end 50.8 54.102) (width 0.25) (layer F.Cu) (net 74))
-  (segment (start 38.1 58.42) (end 46.482 58.42) (width 0.25) (layer F.Cu) (net 74))
+  (segment (start 38.1 58.42) (end 43.434 58.42) (width 0.5) (layer F.Cu) (net 74))
+  (segment (start 50.8 51.054) (end 50.8 31.75) (width 0.5) (layer F.Cu) (net 74))
+  (segment (start 43.434 58.42) (end 50.8 51.054) (width 0.5) (layer F.Cu) (net 74))
   (zone (net 3) (net_name GND) (layer F.Cu) (hatch edge 0.508)
     (connect_pads (clearance 0.508))

Commit message: update,
Parts:
- moved J4 24.3 mm to (24.8, 83.8)
- moved J3 19.9 mm to (19.7, 83.8)
- moved R2 17.2 mm to (27.2, 33.3), turned to 90 degrees
- moved R1 16.8 mm to (27.2, 38.8), turned to 90 degrees
- moved D11 15.2 mm to (62.4, 29.8)
- moved D12 15.2 mm to (71.6, 29.8)
- moved D13 15.2 mm to (80.8, 29.8)
- moved D14 15.2 mm to (90.0, 29.8)
- moved D16 15.2 mm to (108.5, 29.8)
- moved D19 15.2 mm to (62.4, 38.7)
- moved D20 15.2 mm to (71.6, 38.7)
- moved D21 15.2 mm to (80.8, 38.7)
- moved D22 15.2 mm to (90.0, 38.7)
- moved D24 15.2 mm to (108.5, 38.7)
- moved D27 15.2 mm to (62.4, 47.6)
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Routing:
- net VCC: track 845.9 -> 1221.1 mm, vias 9 -> 33
- net Net-(J4-Pad3): track 35.1 -> 54.6 mm
- net /PWM_TO_LED: track 57.9 -> 39.0 mm
- net GND: track 968.6 -> 951.7 mm, vias 11 -> 18
- net V_EXT_LED: track 81.2 -> 87.0 mm
- net +5V: track 14.8 -> 16.4 mm
