File: ws2812-stm32-interface.kicad_pcb (KiCad board)
At the start: 2 copper layers, 100.3 x 76.2 mm, 81 parts, among them J1 Conn_01x03, J2 Conn_01x03, J3 WS2812_DEST, J4 WS2812_SOURCE, U1 74AHCT1G125

Commit message: update,
Parts:
- moved ZD2 2.65 mm to (29.6, 26.8)
Routing:
- net VCC: track 1221.1 -> 1227.8 mm
- net V_EXT_LED: track 87.0 -> 88.6 mm
Changed lines of the file:
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@@
     (thickness 1.6)
     (drawings 5)
-    (tracks 1105)
+    (tracks 1107)
     (zones 0)
     (modules 81)
@@
   )
   (module Diodes_SMD:D_SOD-123F (layer F.Cu)
-    (at 32.26076 26.924571)
+    (at 29.6164 26.7716)
     (descr D_SOD-123F)
     (tags D_SOD-123F)
@@
   (segment (start 18.873328 33.086869) (end 18.873328 29.836869) (width 1) (layer F.Cu) (net 4) (status 30))
   (segment (start 18.873328 29.836869) (end 18.873328 26.586869) (width 1) (layer F.Cu) (net 4) (status 30))
-  (segment (start 28.18076 25.994571) (end 29.11076 26.924571) (width 1) (layer F.Cu) (net 4))
-  (segment (start 28.18076 21.174571) (end 28.18076 25.994571) (width 1) (layer F.Cu) (net 4) (status 10))
-  (segment (start 29.11076 26.924571) (end 30.71075 26.924571) (width 1) (layer F.Cu) (net 4) (status 20))
   (segment (start 54.210571 23.876) (end 55.658571 22.428) (width 1) (layer F.Cu) (net 4))
   (segment (start 46.442 22.428) (end 47.066 22.428) (width 1) (layer F.Cu) (net 4))
@@
   (segment (start 23.746 33.144) (end 25.146 34.544) (width 1) (layer F.Cu) (net 4))
   (segment (start 22.352 33.144) (end 23.746 33.144) (width 1) (layer F.Cu) (net 4))
+  (segment (start 28.18076 21.174571) (end 28.18076 24.384) (width 1) (layer F.Cu) (net 4))
+  (segment (start 28.18076 26.68516) (end 28.2672 26.7716) (width 1) (layer F.Cu) (net 4))
+  (segment (start 28.18076 21.174571) (end 28.18076 26.68516) (width 1) (layer F.Cu) (net 4))
+  (segment (start 28.2164 21.210211) (end 28.18076 21.174571) (width 1) (layer F.Cu) (net 4))
+  (segment (start 28.2164 26.7716) (end 28.2164 21.210211) (width 1) (layer F.Cu) (net 4))
   (segment (start 35.814 29.21) (end 34.925 29.21) (width 0.5) (layer F.Cu) (net 5))
   (segment (start 35.814 29.21) (end 34.29 29.21) (width 0.5) (layer F.Cu) (net 5))
@@
   (segment (start 75.946 21.844) (end 75.946 19.812) (width 0.25) (layer F.Cu) (net 7))
   (segment (start 76.53 22.428) (end 75.946 21.844) (width 0.25) (layer F.Cu) (net 7))
-  (segment (start 33.26076 21.174571) (end 33.26076 24.174571) (width 1) (layer F.Cu) (net 8) (status 10))
-  (segment (start 33.66076 24.574571) (end 33.66076 26.924571) (width 1) (layer F.Cu) (net 8) (status 20))
-  (segment (start 33.26076 24.174571) (end 33.66076 24.574571) (width 1) (layer F.Cu) (net 8))
   (segment (start 19.685 83.82) (end 24.765 83.82) (width 1) (layer B.Cu) (net 8))
   (segment (start 17.145 83.82) (end 19.685 83.82) (width 1) (layer F.Cu) (net 8))
@@
   (segment (start 25.908 52.07) (end 23.876 52.07) (width 1) (layer B.Cu) (net 8))
   (segment (start 33.26076 25.92124) (end 29.464 29.718) (width 1) (layer B.Cu) (net 8))
+  (segment (start 33.26076 21.174571) (end 33.26076 26.32764) (width 1) (layer F.Cu) (net 8))
+  (segment (start 32.8168 26.7716) (end 33.26076 26.32764) (width 1) (layer F.Cu) (net 8))
+  (segment (start 31.0164 26.7716) (end 32.8168 26.7716) (width 1) (layer F.Cu) (net 8))
   (segment (start 27.178 31.924) (end 29.718 31.924) (width 0.25) (layer F.Cu) (net 9))
   (segment (start 27.178 37.432) (end 29.718 37.432) (width 0.25) (layer F.Cu) (net 10))
@@
   (segment (start 35.814 77.216) (end 34.29 78.74) (width 0.5) (layer F.Cu) (net 74))
   (zone (net 3) (net_name GND) (layer F.Cu) (hatch edge 0.508)
-    (connect_pads (clearance 0.254))
+    (connect_pads no (clearance 0.254))
     (min_thickness 0.254)
     (fill yes (arc_segments 16) (thermal_gap 0.508) (thermal_bridge_width 0.508))
