File: ws2812-stm32-interface.sch (KiCad schematic (older format))
At the start: 14 parts, among them J1 Conn_01x03, J2 Conn_01x03, U1 74AHCT1G125

Commit message: update,
Other:
- note added: "LEGEND:\n\n+5V: 5V supply from MCU side,\nV_EXT_LED: 5V power supply from LED strap(if possible)\n\nVDD: joined power supply to LED strap\n"
- note removed: "Assumption:\n\n+5V is supply from MCU side,\nV_EXT_LED is from LED side."
Changed lines of the file:
@@
 Wire Wire Line
 	7100 1400 7100 1500
-Text Notes 950  1700 0    50   ~ 0
-Assumption:\n\n+5V is supply from MCU side,\nV_EXT_LED is from LED side.
+Text Notes 900  2950 0    50   ~ 0
+LEGEND:\n\n+5V:  5V supply from MCU side,\nV_EXT_LED: 5V power supply from LED strap(if possible)\n\nVDD: joined power supply to LED strap\n
 $Comp
 L Connector_Generic:Conn_01x03 J1

Commit message: update,
Parts:
- D1, D2: value mbr120 -> MBR120
- D3: value LED -> GREEN
- D4: value LED -> RED
Changed lines of the file:
@@
 P 2550 1650
 F 0 "D1" V 2596 1571 50  0000 R CNN
-F 1 "mbr120" V 2505 1571 50  0000 R CNN
+F 1 "MBR120" V 2505 1571 50  0000 R CNN
 F 2 "Diodes_SMD:D_SOD-123F" H 2550 1650 50  0001 C CNN
 F 3 "~" H 2550 1650 50  0001 C CNN
@@
 P 3100 1650
 F 0 "D2" V 3146 1571 50  0000 R CNN
-F 1 "mbr120" V 3055 1571 50  0000 R CNN
+F 1 "MBR120" V 3055 1571 50  0000 R CNN
 F 2 "Diodes_SMD:D_SOD-123F" H 3100 1650 50  0001 C CNN
 F 3 "~" H 3100 1650 50  0001 C CNN
@@
 U 1 1 5BBA6D41
 P 4550 1950
-F 0 "D4" V 4588 1833 50  0000 R CNN
-F 1 "LED" V 4497 1833 50  0000 R CNN
+F 0 "D4" V 4588 1832 50  0000 R CNN
+F 1 "RED" V 4497 1832 50  0000 R CNN
 F 2 "LEDs:LED_0805_HandSoldering" H 4550 1950 50  0001 C CNN
 F 3 "~" H 4550 1950 50  0001 C CNN
@@
 U 1 1 5BBA804C
 P 4150 1950
-F 0 "D3" V 4188 1833 50  0000 R CNN
-F 1 "LED" V 4097 1833 50  0000 R CNN
+F 0 "D3" V 4188 1832 50  0000 R CNN
+F 1 "GREEN" V 4097 1832 50  0000 R CNN
 F 2 "LEDs:LED_0805_HandSoldering" H 4150 1950 50  0001 C CNN
 F 3 "~" H 4150 1950 50  0001 C CNN

Commit message: update,
Parts:
- added J3: WS2812_DEST, footprint-lib:Pin_Header_Straight_1x04_Pitch2.54mm, symbol Connector_Generic:Conn_01x04
- added J4: WS2812_SOURCE, footprint-lib:Pin_Header_Straight_1x04_Pitch2.54mm, symbol Connector_Generic:Conn_01x04
- added JP1: Jumper_NC_Dual, footprint-lib:Pin_Header_Straight_1x03_Pitch2.54mm, symbol Device:Jumper_NC_Dual
- LD_O1: renamed from D4; value RED -> ORANGE
- renumbered D3 to LD_G1, D1 to ZD1, D2 to ZD2
Connections:
- wire segments 40 -> 58
