File: ws2812-stm32-interface.sch (KiCad schematic (older format))
At the start: 17 parts, among them J1 Conn_01x03, J2 Conn_01x03, J3 WS2812_DEST, J4 WS2812_SOURCE, U1 74AHCT1G125

Commit message: update,
Parts:
- C1, C2, C3, C4, C5: footprint Capacitors_SMD:C_0805_HandSoldering -> Capacitor_SMD:C_0805_2012Metric_Pad1.15x1.40mm_HandSolder
- J1, JP1: footprint footprint-lib:Pin_Header_Straight_1x03_Pitch2.54mm -> Connector_PinHeader_2.54mm:PinHeader_1x03_P2.54mm_Vertical
- J2: footprint Connectors_Terminal_Blocks:TerminalBlock_bornier-4_P5.08mm -> w_conn_screw:mstbva_2,5-4-g-5,08
- J3, J4: footprint footprint-lib:Pin_Header_Straight_1x04_Pitch2.54mm -> Connector_PinHeader_2.54mm:PinHeader_1x04_P2.54mm_Vertical
- LD_G1, LD_O1: footprint LEDs:LED_0805_HandSoldering -> LED_SMD:LED_0805_2012Metric_Pad1.15x1.40mm_HandSolder
- R1, R2: footprint Resistors_SMD:R_0805_HandSoldering -> Resistor_SMD:R_0805_2012Metric_Pad1.15x1.40mm_HandSolder
- U1: footprint TO_SOT_Packages_SMD:SOT-23-5_HandSoldering -> Package_TO_SOT_SMD:SOT-23-5_HandSoldering
- ZD1, ZD2: footprint Diodes_SMD:D_SOD-123F -> Diode_SMD:D_SOD-123F
Changed lines of the file:
@@
 F 0 "U1" H 4275 3176 50  0000 C CNN
 F 1 "74AHCT1G125" H 4275 3085 50  0000 C CNN
-F 2 "TO_SOT_Packages_SMD:SOT-23-5_HandSoldering" H 4300 3350 50  0001 C CNN
+F 2 "Package_TO_SOT_SMD:SOT-23-5_HandSoldering" H 4300 3350 50  0001 C CNN
 F 3 "http://www.ti.com/lit/sg/scyt129e/scyt129e.pdf" H 4300 3350 50  0001 C CNN
 F 4 "SOD-123FL" H 4300 3350 50  0001 C CNN "Field4"
@@
 F 0 "ZD1" V 2596 1571 50  0000 R CNN
 F 1 "MBR120" V 2505 1571 50  0000 R CNN
-F 2 "Diodes_SMD:D_SOD-123F" H 2550 1650 50  0001 C CNN
+F 2 "Diode_SMD:D_SOD-123F" H 2550 1650 50  0001 C CNN
 F 3 "~" H 2550 1650 50  0001 C CNN
 	1    2550 1650
@@
 F 0 "ZD2" V 3146 1571 50  0000 R CNN
 F 1 "MBR120" V 3055 1571 50  0000 R CNN
-F 2 "Diodes_SMD:D_SOD-123F" H 3100 1650 50  0001 C CNN
+F 2 "Diode_SMD:D_SOD-123F" H 3100 1650 50  0001 C CNN
 F 3 "~" H 3100 1650 50  0001 C CNN
 	1    3100 1650
@@
 F 0 "C1" H 5465 1741 50  0000 L CNN
 F 1 "10u" H 5465 1650 50  0000 L CNN
-F 2 "Capacitors_SMD:C_0805_HandSoldering" H 5388 1500 50  0001 C CNN
+F 2 "Capacitor_SMD:C_0805_2012Metric_Pad1.15x1.40mm_HandSolder" H 5388 1500 50  0001 C CNN
 F 3 "~" H 5350 1650 50  0001 C CNN
 F 4 "0805" H 5465 1559 50  0000 L CNN "Field4"
@@
 F 0 "C2" H 5915 1741 50  0000 L CNN
 F 1 "10u" H 5915 1650 50  0000 L CNN
-F 2 "Capacitors_SMD:C_0805_HandSoldering" H 5838 1500 50  0001 C CNN
+F 2 "Capacitor_SMD:C_0805_2012Metric_Pad1.15x1.40mm_HandSolder" H 5838 1500 50  0001 C CNN
 F 3 "~" H 5800 1650 50  0001 C CNN
 F 4 "0805" H 5915 1559 50  0000 L CNN "Field4"
@@
 F 0 "C3" H 6365 1741 50  0000 L CNN
 F 1 "10u" H 6365 1650 50  0000 L CNN
-F 2 "Capacitors_SMD:C_0805_HandSoldering" H 6288 1500 50  0001 C CNN
+F 2 "Capacitor_SMD:C_0805_2012Metric_Pad1.15x1.40mm_HandSolder" H 6288 1500 50  0001 C CNN
 F 3 "~" H 6250 1650 50  0001 C CNN
 F 4 "0805" H 6365 1559 50  0000 L CNN "Field4"
@@
 F 0 "C4" H 6815 1741 50  0000 L CNN
 F 1 "10u" H 6815 1650 50  0000 L CNN
-F 2 "Capacitors_SMD:C_0805_HandSoldering" H 6738 1500 50  0001 C CNN
+F 2 "Capacitor_SMD:C_0805_2012Metric_Pad1.15x1.40mm_HandSolder" H 6738 1500 50  0001 C CNN
 F 3 "~" H 6700 1650 50  0001 C CNN
 F 4 "0805" H 6815 1559 50  0000 L CNN "Field4"
@@
 F 0 "C5" H 7215 1741 50  0000 L CNN
 F 1 "10u" H 7215 1650 50  0000 L CNN
-F 2 "Capacitors_SMD:C_0805_HandSoldering" H 7138 1500 50  0001 C CNN
+F 2 "Capacitor_SMD:C_0805_2012Metric_Pad1.15x1.40mm_HandSolder" H 7138 1500 50  0001 C CNN
 F 3 "~" H 7100 1650 50  0001 C CNN
 F 4 "0805" H 7215 1559 50  0000 L CNN "Field4"
@@
 F 0 "J1" H 2770 3125 50  0000 C CNN
 F 1 "Conn_01x03" H 2770 3216 50  0000 C CNN
-F 2 "footprint-lib:Pin_Header_Straight_1x03_Pitch2.54mm" H 2850 3450 50  0001 C CNN
+F 2 "Connector_PinHeader_2.54mm:PinHeader_1x03_P2.54mm_Vertical" H 2850 3450 50  0001 C CNN
 F 3 "~" H 2850 3450 50  0001 C CNN
 	1    2850 3450
@@
 F 0 "J2" H 5369 3025 50  0000 C CNN
 F 1 "Conn_01x03" H 5369 3116 50  0000 C CNN
-F 2 "Connectors_Terminal_Blocks:TerminalBlock_bornier-4_P5.08mm" H 5450 3450 50  0001 C CNN
+F 2 "w_conn_screw:mstbva_2,5-4-g-5,08" H 5450 3450 50  0001 C CNN
 F 3 "~" H 5450 3450 50  0001 C CNN
 	1    5450 3450
@@
 F 0 "R2" H 4620 1546 50  0000 L CNN
 F 1 "104" H 4620 1455 50  0000 L CNN
-F 2 "Resistors_SMD:R_0805_HandSoldering" V 4480 1500 50  0001 C CNN
+F 2 "Resistor_SMD:R_0805_2012Metric_Pad1.15x1.40mm_HandSolder" V 4480 1500 50  0001 C CNN
 F 3 "~" H 4550 1500 50  0001 C CNN
 	1    4550 1500
@@
 F 0 "LD_O1" V 4588 1832 50  0000 R CNN
 F 1 "ORANGE" V 4497 1832 50  0000 R CNN
-F 2 "LEDs:LED_0805_HandSoldering" H 4550 1950 50  0001 C CNN
+F 2 "LED_SMD:LED_0805_2012Metric_Pad1.15x1.40mm_HandSolder" H 4550 1950 50  0001 C CNN
 F 3 "~" H 4550 1950 50  0001 C CNN
 	1    4550 1950
@@
 F 0 "R1" H 4220 1546 50  0000 L CNN
 F 1 "104" H 4220 1455 50  0000 L CNN
-F 2 "Resistors_SMD:R_0805_HandSoldering" V 4080 1500 50  0001 C CNN
+F 2 "Resistor_SMD:R_0805_2012Metric_Pad1.15x1.40mm_HandSolder" V 4080 1500 50  0001 C CNN
 F 3 "~" H 4150 1500 50  0001 C CNN
 	1    4150 1500
@@
 F 0 "LD_G1" V 4188 1832 50  0000 R CNN
 F 1 "GREEN" V 4097 1832 50  0000 R CNN
-F 2 "LEDs:LED_0805_HandSoldering" H 4150 1950 50  0001 C CNN
+F 2 "LED_SMD:LED_0805_2012Metric_Pad1.15x1.40mm_HandSolder" H 4150 1950 50  0001 C CNN
 F 3 "~" H 4150 1950 50  0001 C CNN
 	1    4150 1950
@@
 F 0 "J3" H 10169 4375 50  0000 C CNN
 F 1 "WS2812_DEST" H 10169 4466 50  0000 C CNN
-F 2 "footprint-lib:Pin_Header_Straight_1x04_Pitch2.54mm" H 10250 4800 50  0001 C CNN
+F 2 "Connector_PinHeader_2.54mm:PinHeader_1x04_P2.54mm_Vertical" H 10250 4800 50  0001 C CNN
 F 3 "~" H 10250 4800 50  0001 C CNN
 	1    10250 4800
@@
 F 0 "J4" H 6669 4725 50  0000 C CNN
 F 1 "WS2812_SOURCE" H 6669 4816 50  0000 C CNN
-F 2 "footprint-lib:Pin_Header_Straight_1x04_Pitch2.54mm" H 6750 5150 50  0001 C CNN
+F 2 "Connector_PinHeader_2.54mm:PinHeader_1x04_P2.54mm_Vertical" H 6750 5150 50  0001 C CNN
 F 3 "~" H 6750 5150 50  0001 C CNN
 	1    6750 5150
@@
 F 0 "JP1" V 7846 4552 50  0000 L CNN
 F 1 "Jumper_NC_Dual" V 7755 4552 50  0000 L CNN
-F 2 "footprint-lib:Pin_Header_Straight_1x03_Pitch2.54mm" H 7800 4450 50  0001 C CNN
+F 2 "Connector_PinHeader_2.54mm:PinHeader_1x03_P2.54mm_Vertical" H 7800 4450 50  0001 C CNN
 F 3 "~" H 7800 4450 50  0001 C CNN
 	1    7800 4450
