File: led_array.sch (KiCad schematic (older format))
At the start: 64 parts

Commit message: update,
Parts:
- D1, D10, D11, D12, D13, D14, D15, D16, D17, D18, D19, D2, D20, D21, D22, D23, D24, D25, D26, D27, D28, D29, D3, D30, D31, D32, D33, D34, D35, D36, D37, D38, D39, D4, D40, D41, D42, D43, D44, D45, D46, D47, D48, D49, D5, D50, D51, D52, D53, D54, D55, D56, D57, D58, D59, D6, D60, D61, D62, D63, D64, D7, D8, D9: footprint LEDs:LED_WS2812B-PLCC4 -> footprint-lib:LED_WS2812B_PLCC4_5.0x5.0mm_P3.2mm

Commit message: update,
Parts:
- removed D1, D10, D13, D14, D15, D16, D25, D26, D27, D28, D33, D34, D35, D37, D38, D4, D41, D43, D44, D45, D46, D51, D9: WS2812B, footprint-lib:LED_WS2812B_PLCC4_5.0x5.0mm_P3.2mm, symbol LED:WS2812B
- added D513, D516, D521, D522, D525, D526, D527, D528, D537, D538, D539, D540, D545, D546, D547, D549, D550, D553, D555, D556, D557, D558, D563: WS2812B, footprint-lib:LED_WS2812B_PLCC4_5.0x5.0mm_P3.2mm, symbol LED:WS2812B
- renumbered D2 to D514, D3 to D515, D5 to D517, D6 to D518, D7 to D519, D8 to D520, D11 to D523, D12 to D524, D17 to D529, D18 to D530, D19 to D531, D20 to D532, D21 to D533, D22 to D534, D23 to D535, D24 to D536, D29 to D541, D30 to D542, D31 to D543, D32 to D544, D36 to D548, D39 to D551, D40 to D552, D42 to D554, D47 to D559, D48 to D560, D49 to D561, D50 to D562, D52 to D564, D53 to D565, D54 to D566, D55 to D567, D56 to D568, D57 to D569, D58 to D570, D59 to D571, D60 to D572, D61 to D573, D62 to D574, D63 to D575, D64 to D576
